Commit message: added d415 cam instead of all sensors pkg

File: starbots_ur3e/ur_description/urdf/ur.urdf.xacro (robot description, xacro)
@@ -7,5 +7,6 @@
    <!--<xacro:include filename="$(find robotiq_85_description)/urdf/robotiq_85_gripper_macro_gz.urdf.xacro" />-->
    <xacro:include filename="$(find rg2_gripper_description)/urdf/rg2_gripper.urdf.xacro" />
-   <xacro:include filename="$(find robotnik_sensors)/urdf/all_sensors.urdf.xacro" />
+   <xacro:include filename="$(find ur_description)/urdf/intel_d415.urdf.xacro" />
+   <!-- <xacro:include filename="$(find robotnik_sensors)/urdf/all_sensors.urdf.xacro" /> -->
    <!-- possible 'ur_type' values: ur3, ur3e, ur5, ur5e, ur10, ur10e, ur16e -->
    <!-- the default value should raise an error in case this was called without defining the type -->
@@ -88,17 +89,19 @@
      <origin xyz="0 0 0" rpy="0 0 0" />          <!-- position robot in the world -->
    </xacro:ur_robot>
-   <!--<xacro:robotiq_85_gripper prefix="" parent="tool0" >
+   <!-- <xacro:robotiq_85_gripper prefix="" parent="tool0" >
        <origin xyz="0.0 0 0.0" rpy="0 -1.57 1.57"/>
-   </xacro:robotiq_85_gripper>-->
+   </xacro:robotiq_85_gripper> -->
    <xacro:rg2_gripper prefix="rg2_gripper" parent="tool0" >
        <!--<origin xyz="0.0 0 0.0" rpy="0 -1.57 1.57"/>-->
    </xacro:rg2_gripper>
-   <xacro:sensor_r430 prefix="wrist_rgbd" parent="base_link" >
-       <!-- <origin xyz="-0.2 -0.3 0.2" rpy="0 ${pi/3} ${pi/2}"/> -->
-       <origin xyz="-0.25 -0.3 0.2" rpy="0 ${pi/3} ${pi/2}"/>
-   </xacro:sensor_r430>
-    <xacro:sensor_r430 prefix="camera" parent="base_link" >
-       <origin xyz="0.8 0.5 0.2" rpy="0 ${pi/6} ${pi}"/>
-   </xacro:sensor_r430>
+   <xacro:sensor_d415
+        name="D415"
+        parent="base_link"
+        flag_color="1"
+        flag_ir="1"
+        flag_depth="1"
+        updaterate="30" >
+        <origin xyz="0.5 0.75 0.1" rpy="0 ${pi/6} ${-pi/2}"/>
+    </xacro:sensor_d415>
    <xacro:if value="$(arg sim_gazebo)">
     <!-- Gazebo plugins -->

File: starbots_ur3e/ur_description/urdf/ur_moveit.urdf.xacro (robot description, xacro)
@@ -5,6 +5,8 @@
    <!-- import main macro -->
    <xacro:include filename="$(find ur_description)/urdf/ur_macro.xacro"/>
-   <xacro:include filename="$(find robotiq_85_description)/urdf/robotiq_85_gripper_macro_gz.urdf.xacro" />
-   <xacro:include filename="$(find robotnik_sensors)/urdf/all_sensors.urdf.xacro" />
+   <!-- <xacro:include filename="$(find robotiq_85_description)/urdf/robotiq_85_gripper_macro_gz.urdf.xacro" /> -->
+   <xacro:include filename="$(find rg2_gripper_description)/urdf/rg2_gripper.urdf.xacro" />
+   <xacro:include filename="$(find ur_description)/urdf/intel_d415.urdf.xacro" />
+   <!-- <xacro:include filename="$(find robotnik_sensors)/urdf/all_sensors.urdf.xacro" /> -->
    <!-- possible 'ur_type' values: ur3, ur3e, ur5, ur5e, ur10, ur10e, ur16e -->
    <!-- the default value should raise an error in case this was called without defining the type -->
@@ -109,11 +111,19 @@
      <origin xyz="0 0 0" rpy="0 0 0" />          <!-- position robot in the world -->
    </xacro:ur_robot>
-   <xacro:robotiq_85_gripper prefix="" parent="tool0" >
+   <!-- <xacro:robotiq_85_gripper prefix="" parent="tool0" >
        <origin xyz="0.0 0 0.0" rpy="0 -1.57 1.57"/>
-   </xacro:robotiq_85_gripper>
-   <xacro:sensor_r430 prefix="wrist_rgbd" parent="base_link" >
-       <!--<origin xyz="0.35 0.45 0.1" rpy="0 ${pi/6} ${-pi/2}"/>-->
-       <origin xyz="0.5 0.75 0.1" rpy="0 ${pi/6} ${-pi/2}"/>
-   </xacro:sensor_r430>
+   </xacro:robotiq_85_gripper> -->
+   <xacro:rg2_gripper prefix="rg2_gripper" parent="tool0" >
+       <!--<origin xyz="0.0 0 0.0" rpy="0 -1.57 1.57"/>-->
+   </xacro:rg2_gripper>
+    <xacro:sensor_d415
+        name="D415"
+        parent="base_link"
+        flag_color="1"
+        flag_ir="1"
+        flag_depth="1"
+        updaterate="30" >
+        <origin xyz="0.5 0.75 0.1" rpy="0 ${pi/6} ${-pi/2}"/>
+    </xacro:sensor_d415>
    <xacro:if value="$(arg sim_gazebo)">
     <!-- Gazebo plugins -->

Commit message: setup changed for new gripper

File: starbots_ur3e/ur_description/urdf/ur.urdf.xacro (robot description, xacro)
@@ -5,6 +5,6 @@
    <!-- import main macro -->
    <xacro:include filename="$(find ur_description)/urdf/ur_macro.xacro"/>
-   <!--<xacro:include filename="$(find robotiq_85_description)/urdf/robotiq_85_gripper_macro_gz.urdf.xacro" />-->
-   <xacro:include filename="$(find rg2_gripper_description)/urdf/rg2_gripper.urdf.xacro" />
+   <xacro:include filename="$(find robotiq_85_description)/urdf/robotiq_85_gripper_macro_gz.urdf.xacro" />
+   <!-- <xacro:include filename="$(find rg2_gripper_description)/urdf/rg2_gripper.urdf.xacro" /> -->
    <xacro:include filename="$(find ur_description)/urdf/intel_d415.urdf.xacro" />
    <!-- <xacro:include filename="$(find robotnik_sensors)/urdf/all_sensors.urdf.xacro" /> -->
@@ -89,11 +89,11 @@
      <origin xyz="0 0 0" rpy="0 0 0" />          <!-- position robot in the world -->
    </xacro:ur_robot>
-   <!-- <xacro:robotiq_85_gripper prefix="" parent="tool0" >
+   <xacro:robotiq_85_gripper prefix="" parent="tool0" >
+       <origin xyz="0.0 0.0 0.0" rpy="0 -1.57 1.57"/>
+   </xacro:robotiq_85_gripper>
+   <!-- <xacro:rg2_gripper prefix="rg2_gripper" parent="tool0" >
        <origin xyz="0.0 0 0.0" rpy="0 -1.57 1.57"/>
-   </xacro:robotiq_85_gripper> -->
-   <xacro:rg2_gripper prefix="rg2_gripper" parent="tool0" >
-       <!--<origin xyz="0.0 0 0.0" rpy="0 -1.57 1.57"/>-->
-   </xacro:rg2_gripper>
-   <xacro:sensor_d415
+   </xacro:rg2_gripper> -->
+   <!-- <xacro:sensor_d415
         name="D415"
         parent="base_link"
@@ -103,5 +103,5 @@
         updaterate="30" >
         <origin xyz="0.5 0.75 0.1" rpy="0 ${pi/6} ${-pi/2}"/>
-    </xacro:sensor_d415>
+    </xacro:sensor_d415> -->
    <xacro:if value="$(arg sim_gazebo)">
     <!-- Gazebo plugins -->

File: starbots_ur3e/ur_description/urdf/ur_moveit.urdf.xacro (robot description, xacro)
@@ -5,6 +5,6 @@
    <!-- import main macro -->
    <xacro:include filename="$(find ur_description)/urdf/ur_macro.xacro"/>
-   <!-- <xacro:include filename="$(find robotiq_85_description)/urdf/robotiq_85_gripper_macro_gz.urdf.xacro" /> -->
-   <xacro:include filename="$(find rg2_gripper_description)/urdf/rg2_gripper.urdf.xacro" />
+   <xacro:include filename="$(find robotiq_85_description)/urdf/robotiq_85_gripper_macro_gz.urdf.xacro" />
+   <!-- <xacro:include filename="$(find rg2_gripper_description)/urdf/rg2_gripper.urdf.xacro" /> -->
    <xacro:include filename="$(find ur_description)/urdf/intel_d415.urdf.xacro" />
    <!-- <xacro:include filename="$(find robotnik_sensors)/urdf/all_sensors.urdf.xacro" /> -->
@@ -111,11 +111,11 @@
      <origin xyz="0 0 0" rpy="0 0 0" />          <!-- position robot in the world -->
    </xacro:ur_robot>
-   <!-- <xacro:robotiq_85_gripper prefix="" parent="tool0" >
-       <origin xyz="0.0 0 0.0" rpy="0 -1.57 1.57"/>
-   </xacro:robotiq_85_gripper> -->
-   <xacro:rg2_gripper prefix="rg2_gripper" parent="tool0" >
-       <!--<origin xyz="0.0 0 0.0" rpy="0 -1.57 1.57"/>-->
-   </xacro:rg2_gripper>
-    <xacro:sensor_d415
+   <xacro:robotiq_85_gripper prefix="" parent="tool0" >
+       <origin xyz="0.0 0.0 0.0" rpy="0 -1.57 1.57"/>
+   </xacro:robotiq_85_gripper>
+   <!-- <xacro:rg2_gripper prefix="rg2_gripper" parent="tool0" > -->
+       <!-- <origin xyz="0.0 0 0.0" rpy="0 -1.57 1.57"/> -->
+   <!-- </xacro:rg2_gripper> -->
+    <!-- <xacro:sensor_d415
         name="D415"
         parent="base_link"
@@ -125,5 +125,5 @@
         updaterate="30" >
         <origin xyz="0.5 0.75 0.1" rpy="0 ${pi/6} ${-pi/2}"/>
-    </xacro:sensor_d415>
+    </xacro:sensor_d415> -->
    <xacro:if value="$(arg sim_gazebo)">
     <!-- Gazebo plugins -->
